File: UINIO-MCU-HC32F460PETB.kicad_pcb (KiCad board)
At the start: 2 copper layers, 93.7 x 53.1 mm, 55 parts, among them J1 Conn_01x18_Pin, J2 Conn_01x34_Pin, J3 Conn_01x34_Pin, J4 MD, J5 Conn_01x04_Pin, J6 Conn_01x04_Pin, J7 Conn_01x05_Pin, J8 Conn_01x04_Pin, J9 Conn_01x04_Pin, SW1 NRST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

Commit message: update
Parts:
- moved C7 21.7 mm to (129.3, 93.6), turned to -90 degrees
- moved C4 21.2 mm to (134.6, 93.6), turned to -90 degrees
- moved U1 21.2 mm to (132.0, 93.6), turned to 90 degrees
- moved R3 3.54 mm to (121.6, 93.6), turned to -90 degrees
- moved D1 2.70 mm to (119.3, 93.5), turned to 90 degrees
- moved R6 1.87 mm to (131.4, 107.2)
- moved R7 1.87 mm to (128.9, 107.2)
- moved C10 1.82 mm to (115.2, 85.8)
- moved C11 1.82 mm to (117.3, 85.8)
- moved C23 1.82 mm to (117.3, 116.3)
- moved C24 1.82 mm to (115.2, 116.3)
- moved R1 1.76 mm to (119.8, 99.8)
- moved R2 1.76 mm to (119.8, 102.8)
- moved C19 0.19 mm to (160.5, 114.0)
- moved C9 0.19 mm to (150.0, 115.5)
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Connections:
- J7 pad 2: /PA14/JTCK_SWCLK -> /NRST
- J7 pad 3: /PA13/JTMS_SWDIO -> /PA14/JTCK_SWCLK
- J7 pad 4: /NRST -> /PA13/JTMS_SWDIO

Commit message: update
Parts:
- moved C10 2.09 mm to (117.3, 85.8)
- moved C11 2.09 mm to (115.2, 85.8)
- moved C19 0.78 mm to (159.7, 114.0)
- moved U1 0.18 mm to (131.9, 93.4)
- moved C12 0.11 mm to (150.5, 85.9)
- moved C8 0.10 mm to (147.5, 85.9)
Routing:
- net VCC_3.3V: track 0.00 -> 78.2 mm, vias 0 -> 3
- net VCC_5V: track 0.00 -> 49.8 mm, vias 0 -> 2
- net /PA14/JTCK_SWCLK: track 0.00 -> 33.3 mm
- net /PA13/JTMS_SWDIO: track 0.00 -> 10.0 mm
- net Net-(USB1-CC2): track 0.00 -> 7.92 mm
- net Net-(USB1-CC1): track 0.00 -> 7.92 mm
- net Net-(U2-VCAP_1): track 0.00 -> 7.26 mm
- net Net-(D1-A): track 0.00 -> 2.21 mm
- net GND: track 0.00 -> 1.73 mm

Commit message: update
Parts:
- moved C6 3.20 mm to (137.4, 110.3)
- moved L1 3.08 mm to (166.3, 85.9)
- moved L2 3.08 mm to (161.1, 85.9)
- moved C1 3.07 mm to (162.8, 85.9)
- moved C2 3.07 mm to (164.5, 85.9)
- moved C5 1.97 mm to (173.3, 88.4)
- moved C3 1.97 mm to (173.3, 86.7)
- moved L3 1.97 mm to (173.3, 91.9)
- moved L4 1.97 mm to (173.3, 90.2)
- moved C12 1.82 mm to (148.7, 85.9)
- moved C22 1.62 mm to (137.4, 106.1)
- moved C19 1.55 mm to (161.3, 114.0), turned to 180 degrees
- moved C20 1.03 mm to (173.3, 107.8), turned to 180 degrees
- moved HOLE** 1.00 mm to (188.3, 85.6)
- moved HOLE** 1.00 mm to (188.3, 116.6)
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Routing:
- net VCC_3.3V: track 78.2 -> 177.6 mm, vias 3 -> 14
- net /NRST: track 0.00 -> 73.7 mm, vias 0 -> 2
- net /PD15: track 0.00 -> 53.9 mm
- net /PC6: track 0.00 -> 52.0 mm
- net /PD14: track 0.00 -> 51.1 mm
- net /PC7: track 0.00 -> 50.4 mm
- net /PC8: track 0.00 -> 48.8 mm
- net /PD13: track 0.00 -> 48.4 mm
- net VCC_5V: track 49.8 -> 1.49 mm, vias 2 -> 4
- net /PC9: track 0.00 -> 47.2 mm
- net /PA3: track 0.00 -> 46.0 mm
- net /PA12: track 0.00 -> 45.9 mm
- net /PA11: track 0.00 -> 45.7 mm
- net /PA8: track 0.00 -> 45.6 mm
- net /PD12: track 0.00 -> 45.6 mm
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- added copper zone on B.Cu, net GND
- added copper zone on F.Cu, net GND
- added copper zone on B.Cu, net VCC_5V
- added copper zone on F.Cu, net VCC_5V

Commit message: update
Parts:
- moved C16 1.20 mm to (173.3, 112.4)
- moved Y1 1.20 mm to (174.2, 115.1)
- moved C15 1.20 mm to (171.5, 114.2)
Routing:
- net /PE6: track 0.00 -> 48.4 mm
- net /PC13: track 0.00 -> 48.4 mm
- net /PH2: track 0.00 -> 47.5 mm
- net /PE5: track 0.00 -> 45.6 mm
- net /PE4: track 0.00 -> 44.7 mm
- net /PE3: track 0.00 -> 44.0 mm
- net Net-(U2-PC14/XTAL32_OUT): track 19.4 -> 18.8 mm
- net VCC_3.3V: track 177.6 -> 178.2 mm
- net Net-(U2-PC15/XTAL32_IN): track 19.8 -> 19.2 mm
- net GND: vias 148 -> 157
- added copper zone on B.Cu, net VCC_3.3V
- added copper zone on F.Cu, net VCC_3.3V

Commit message: update
Parts:
- J7: value Conn_01x05_Pin -> Conn_01x04_Pin; footprint Connector_PinHeader_2.54mm:PinHeader_1x05_P2.54mm_Vertical -> Connector_PinHeader_2.54mm:PinHeader_1x04_P2.54mm_Vertical
- moved C2 3.79 mm to (160.8, 85.9)
- moved L2 3.13 mm to (164.2, 85.9)
- moved J7 2.54 mm to (134.0, 118.0)
- moved C1 0.33 mm to (162.5, 85.9)
- moved L1 0.33 mm to (165.9, 85.9)
Connections:
- J7 pad 2: /NRST -> /PA14/JTCK_SWCLK
- J7 pad 3: /PA14/JTCK_SWCLK -> /PA13/JTMS_SWDIO
- J7 pad 4: /PA13/JTMS_SWDIO -> VCC_3.3V
- SW1 pad 1: VCC_3.3V -> /NRST
- SW1 pad 2: VCC_3.3V -> /NRST
Routing:
- net VCC_3.3V: track 178.2 -> 320.7 mm, vias 14 -> 19
- net /AVCC: track 0.00 -> 86.0 mm
- net /PA13/JTMS_SWDIO: track 0.00 -> 46.3 mm
- net /PA14/JTCK_SWCLK: track 1.09 -> 40.7 mm, vias 0 -> 1
- net /VREFH: track 0.00 -> 39.5 mm
- net /AVSS: track 0.00 -> 38.6 mm
- net /AVSS/VREFL: track 0.00 -> 37.8 mm
- net /NRST: track 73.7 -> 78.3 mm, vias 2 -> 3
- net GND: track 3.55 -> 5.77 mm, vias 157 -> 220
- net /PB11/MD: track 18.1 -> 16.2 mm
- net /PA1: track 43.9 -> 43.2 mm
- net /PA0: track 44.8 -> 44.2 mm
- net /PA3: track 46.0 -> 45.4 mm
- net /PA2: track 44.7 -> 44.1 mm
- net /PD0: track 19.3 -> 18.8 mm
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
Commit message: update
Routing:
- net VCC_3.3V: vias 19 -> 18
Changed lines of the file:
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@@
-	)
-	(via
-		(at 137.395 84.31)
-		(size 0.7)
-		(drill 0.3)
-		(layers "F.Cu" "B.Cu")
-		(net 70)
 	)
 	(via

Commit message: update
Parts:
- moved R5 1.42 mm to (136.1, 85.4), turned to -90 degrees
- moved C13 1.42 mm to (137.5, 85.4), turned to 90 degrees
- moved SW1 1.33 mm to (132.4, 85.7), turned to 0 degrees
Routing:
- net VCC_3.3V: track 320.7 -> 331.5 mm, vias 18 -> 19
- net /NRST: track 78.3 -> 81.3 mm, vias 3 -> 2
- net GND: track 5.77 -> 5.75 mm, vias 220 -> 224

Commit message: update
Routing:
- net VCC_3.3V: track 331.5 -> 332.8 mm
