File: UINIO-MCU-HC32F460PETB.kicad_pcb (KiCad board)
At the start: 2 copper layers, 93.7 x 53.1 mm, 55 parts, among them J1 Conn_01x18_Pin, J2 Conn_01x34_Pin, J3 Conn_01x34_Pin, J4 MD, J5 Conn_01x04_Pin, J6 Conn_01x04_Pin, J7 Conn_01x04_Pin, J8 Conn_01x04_Pin, J9 Conn_01x04_Pin, SW1 NRST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

Commit message: update
Parts:
- removed J4: MD, Connector_PinHeader_2.54mm:PinHeader_1x02_P2.54mm_Vertical
- added J10: Conn_01x03_Pin, Connector_PinHeader_2.54mm:PinHeader_1x03_P2.54mm_Vertical, F.Cu at (151.8, 118.0)
Routing:
- net VCC_5V: track 1.49 -> 6.89 mm, vias 8 -> 10
- net /PD1: track 20.3 -> 22.6 mm
- net /PD0: track 18.8 -> 21.1 mm
- net /PC12: track 19.9 -> 20.7 mm
- net VCC_3.3V: track 332.8 -> 332.2 mm
- net GND: vias 224 -> 221

Commit message: update
Parts:
- removed J10: Conn_01x03_Pin, Connector_PinHeader_2.54mm:PinHeader_1x03_P2.54mm_Vertical
- added J4: Conn_01x03_Pin, Connector_PinHeader_2.54mm:PinHeader_1x03_P2.54mm_Vertical, F.Cu at (151.8, 118.0)
Routing:
- net GND: vias 221 -> 225
