File: UINIO-MCU-HC32F460PETB.kicad_pcb (KiCad board)
At the start: 2 copper layers, 93.7 x 53.1 mm, 55 parts, among them J1 Conn_01x18_Pin, J2 Conn_01x34_Pin, J3 Conn_01x34_Pin, J4 Conn_01x03_Pin, J5 Conn_01x04_Pin, J6 Conn_01x04_Pin, J7 Conn_01x04_Pin, J8 Conn_01x04_Pin, J9 Conn_01x04_Pin, SW1 NRST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

Commit message: update
Parts:
- added F1: Fuse, Fuse:Fuse_1206_3216Metric, F.Cu at (119.8, 85.0)
Connections:
- J5 pad 1: VCC_5V -> Net-(J5-Pin_1)
- J5 pad 2: VCC_5V -> Net-(J5-Pin_1)
- J5 pad 3: VCC_5V -> Net-(J5-Pin_1)
- J5 pad 4: VCC_5V -> Net-(J5-Pin_1)
Routing:
- net GND: vias 225 -> 228
- added copper zone on F.Cu, net Net-(J5-Pin_1)
Other:
- board text added: "MD/PB11"
- board text added: "UINIO-MCU-HC32F460KETA"
- board text added: "UinIO.com"
- board text added: "Version 1.0.0"
- board text removed: "MD"

Commit message: update
Parts:
- moved R6 3.16 mm to (130.8, 110.3), turned to 180 degrees
- moved R7 2.49 mm to (130.8, 108.7), turned to 0 degrees
- moved C10 2.16 mm to (115.1, 85.8)
- moved C11 2.16 mm to (113.0, 85.8)
- moved C23 2.16 mm to (115.1, 116.3)
- moved C24 2.16 mm to (113.0, 116.3)
- moved F1 2.16 mm to (117.6, 85.0)
- moved J7 1.01 mm to (132.9, 118.0)
- moved R1 0.41 mm to (119.4, 99.8)
- moved R2 0.41 mm to (119.4, 102.8)
Connections:
- J7 pad 1: GND -> VCC_3.3V
- J7 pad 2: /PA14/JTCK_SWCLK -> GND
- J7 pad 3: /PA13/JTMS_SWDIO -> /PA14/JTCK_SWCLK
- J7 pad 4: VCC_3.3V -> /PA13/JTMS_SWDIO
Routing:
- net VCC_3.3V: track 332.2 -> 322.4 mm, vias 19 -> 16
- net /PA13/JTMS_SWDIO: track 46.3 -> 52.6 mm
- net /PA14/JTCK_SWCLK: track 40.7 -> 44.3 mm
- net GND: vias 228 -> 231
Other:
- board text added: "SWD"
- board text added: "UINIO-MCU-HC32F460PETB"
- board text removed: "UINIO-MCU-HC32F460KETA"
