File: UINIO-MCU-HC32F460PETB.kicad_sch (KiCad schematic)
At the start: 44 parts, among them J1 Conn_01x14_Pin, J2 Conn_01x24_Pin, J3 Conn_01x24_Pin, J4 MD, J5 Conn_01x04_Pin, J6 Conn_01x04_Pin, SW1 NRST, U1 ME6211C33M5G, U2 HC32F460KETA-LQFP64, U3 HC32F460PETB-LQFP100, Y1 32.768KHz, Y2 8MHz

Commit message: update
Parts:
- removed U2: HC32F460KETA-LQFP64, Uinio:LQFP-64_L10.0-W10.0-P0.50-LS12.0-BL, symbol Uinio:HC32F460KETA-LQFP64
- added C20, C21, C22: 0.1uF, Capacitor_SMD:C_0603_1608Metric, symbol Device:C
- added J7, J8: Conn_01x38_Pin, symbol Connector:Conn_01x38_Pin
- renumbered U3 to U2
Connections:
- net AVCC: now also U2.22 (AVCC), U2.28 (AVCC)
- net AVCC/VREFH: no longer L4.2
- net AVSS: now also U2.27 (AVSS)
- net AVSS/VREFL: now also U2.20 (AVSS/VREFL)
- net GND: now also U2.10 (VSS), C20.1, C21.1, C22.1
- net PA0: now also U2.23 (PA0/ADC1_IN0)
- net PA1: now also U2.24 (PA1/ADC1_IN1)
- net PA10: now also U2.69 (PA10/USBFS_ID)
- net PA11: now also U2.70 (PA11/USBFS_DM)
- net PA12: now also U2.71 (PA12/USBFS_DP)
- net PA13/JTMS_SWDIO: now also U2.72 (PA13/JTMS_SWDIO)
- net PA14/JTCK_SWCLK: now also U2.76 (PA14/JTCK_SWCLK)
- net PA15: now also U2.77 (PA15/JTDI)
- net PA2: now also U2.25 (PA2/ADC1_IN2)
- net PA3: now also U2.26 (PA3/ADC1_IN3)
- net PA4: now also U2.29 (PA4/ADC12_IN4)
- net PA5: now also U2.30 (PA5/ADC12_IN5)
- net PA6: now also U2.31 (PA6/ADC12_IN6)
- net PA7: now also U2.32 (PA7/ADC12_IN7)
- net PA8: now also U2.67 (PA8)
- net PA9: now also U2.68 (PA9/USBFS_VBUS)
- net PB0: now also U2.35 (PB0/ADC12_IN8)
- net PB1: now also U2.36 (PB1/ADC12_IN9)
- net PB10: now also U2.47 (PB10)
- net PB12: now also U2.51 (PB12)
- net PB13: now also U2.52 (PB13)
- net PB14: now also U2.53 (PB14)
- net PB15: now also U2.54 (PB15)
- net PB2: now also U2.37 (PB2/PVD2EXINP)
- net PB3: now also U2.89 (PB3/JTDO_TRACESWO)
- net PB4: now also U2.90 (PB4/NJTRST)
- net PB5: now also U2.91 (PB5)
- net PB6: now also U2.92 (PB6)
- net PB7: now also U2.93 (PB7)
- net PB8: now also U2.95 (PB8)
- net PB9: now also U2.96 (PB9)
- net PC0: now also U2.15 (PC0/ADC12_IN10)
- net PC1: now also U2.16 (PC1/ADC12_IN11)
- net PC10: now also U2.78 (PC10)
- net PC11: now also U2.79 (PC11)
- net PC12: now also U2.80 (PC12)
- net PC13: now also U2.7 (PC13)
- net PC2: now also U2.17 (PC2/ADC1_IN12)
- net PC3: now also U2.18 (PC3/ADC1_IN13)
- net PC4: now also U2.33 (PC4/ADC1_IN14)
- net PC5: now also U2.34 (PC5/ADC1_IN15)
- net PC6: now also U2.63 (PC6)
- net PC7: now also U2.64 (PC7)
- net PC8: now also U2.65 (PC8)
- net PC9: now also U2.66 (PC9)
- net PD2: now also U2.83 (PD2)
- net PH2: now also U2.6 (PH2)
- net VCC_3.3V: now also U2.11 (VCC), U2.19 (VCC), C20.2, C21.2
- net PE2: now reaches U2.1 (PE2)
- net PE3: now reaches U2.2 (PE3)
- net VREFH: now reaches U2.21 (VREFH)
- net VREFH: now also L4.2
- net PE4: now reaches U2.3 (PE4)
- net PE7: now reaches U2.38 (PE7)
- net PE8: now reaches U2.39 (PE8)
- net PE5: now reaches U2.4 (PE5)
- net PE9: now reaches U2.40 (PE9)
- net PE10: now reaches U2.41 (PE10)
- net PE11: now reaches U2.42 (PE11)
- net PE12: now reaches U2.43 (PE12)
- net PE13: now reaches U2.44 (PE13)
- net PE14: now reaches U2.45 (PE14)
- net PE15: now reaches U2.46 (PE15)
- net PE6: now reaches U2.5 (PE6)
- net PD8: now reaches U2.55 (PD8)
- net PD9: now reaches U2.56 (PD9)
- net PD10: now reaches U2.57 (PD10)
- net PD11: now reaches U2.58 (PD11)
- net PD12: now reaches U2.59 (PD12)
- net PD13: now reaches U2.60 (PD13)
- net PD14: now reaches U2.61 (PD14)
- net PD15: now reaches U2.62 (PD15)
- net at U2.73 (VCAP_2): now also C22.2
- net PD0: now reaches U2.81 (PD0)
- net PD1: now reaches U2.82 (PD1)
- net PD3: now reaches U2.84 (PD3)
- net PD4: now reaches U2.85 (PD4)
- net PD5: now reaches U2.86 (PD5)
- net PD6: now reaches U2.87 (PD6)
- net PD7: now reaches U2.88 (PD7)
- net PE0: now reaches U2.97 (PE0)
- net PE1: now reaches U2.98 (PE1)
Other:
- note added: "38Pin 2.54mm 杜邦排针"
- note added: "HC32F460PETB-LQFP100 最小系统"
- note removed: "32Pin 2.54mm 杜邦排针"
- note removed: "HC32F460KETA-LQFP64 最小系统"
- moved on the sheet: C1, C10, C11, C12, C13, C14, C15, C16, C17, C18, C19, C2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

Commit message: Update
Parts:
- removed J1: Conn_01x14_Pin, Connector_PinHeader_2.54mm:PinHeader_1x14_P2.54mm_Vertical, symbol Connector:Conn_01x14_Pin
- removed J2, J3: Conn_01x24_Pin, Connector_PinHeader_2.54mm:PinHeader_1x24_P2.54mm_Vertical, symbol Connector:Conn_01x24_Pin
- removed J5: Conn_01x04_Pin, Connector_PinHeader_2.54mm:PinHeader_1x04_P2.54mm_Vertical, symbol Connector:Conn_01x04_Pin
- removed J7, J8: Conn_01x38_Pin, symbol Connector:Conn_01x38_Pin
- added C23: 0.1uF, Capacitor_SMD:C_0603_1608Metric, symbol Device:C
- added C24: 1uF, Capacitor_SMD:C_0603_1608Metric, symbol Device:C
- added J1: Conn_01x18_Pin, symbol Connector:Conn_01x18_Pin
- added J10: Conn_01x25_Pin, symbol Connector:Conn_01x25_Pin
- added J2, J3: Conn_01x34_Pin, symbol Connector:Conn_01x34_Pin
- added J5, J6: Conn_01x08_Pin, symbol Connector:Conn_01x08_Pin
- added J8: Conn_01x04_Pin, Connector:FanPinHeader_1x03_P2.54mm_Vertical, symbol Connector:Conn_01x04_Pin
- added J9: Conn_01x04_Pin, symbol Connector:Conn_01x04_Pin
- renumbered J6 to J7
Connections:
- net AVCC: now also J1.4 (Pin_4), J3.32 (Pin_32)
- net AVSS: now also J3.33 (Pin_33)
- net AVSS/VREFL: now also J1.6 (Pin_6)
- net GND: now also C23.1, C24.1, J2.34 (Pin_34), J6.1 (Pin_1), J6.2 (Pin_2), J6.3 (Pin_3), J6.4 (Pin_4), J6.5 (Pin_5), J6.6 (Pin_6), J6.7 (Pin_7), J6.8 (Pin_8), J9.1 (Pin_1), J9.2 (Pin_2), J9.3 (Pin_3), J9.4 (Pin_4)
- net NRST: now also J1.11 (Pin_11)
- net PA0: now also J1.3 (Pin_3)
- net PA1: now also J1.2 (Pin_2)
- net PA10: now also J2.7 (Pin_7)
- net PA11: now also J2.8 (Pin_8)
- net PA12: now also J2.9 (Pin_9)
- net PA13/JTMS_SWDIO: now also J2.10 (Pin_10)
- net PA14/JTCK_SWCLK: now also J2.11 (Pin_11)
- net PA15: now also J2.12 (Pin_12)
- net PA2: now also J1.1 (Pin_1)
- net PA3: now also J3.34 (Pin_34)
- net PA4: now also J3.31 (Pin_31)
- net PA5: now also J3.30 (Pin_30)
- net PA6: now also J3.29 (Pin_29)
- net PA7: now also J3.28 (Pin_28)
- net PA8: now also J2.5 (Pin_5)
- net PA9: now also J2.6 (Pin_6)
- net PB0: now also J3.25 (Pin_25)
- net PB1: now also J3.24 (Pin_24)
- net PB10: now also J3.13 (Pin_13)
- net PB12: now also J3.12 (Pin_12)
- net PB13: now also J3.11 (Pin_11)
- net PB14: now also J3.10 (Pin_10)
- net PB15: now also J3.9 (Pin_9)
- net PB2: now also J3.23 (Pin_23)
- net PB3: now also J2.24 (Pin_24)
- net PB4: now also J2.25 (Pin_25)
- net PB5: now also J2.26 (Pin_26)
- net PB6: now also J2.27 (Pin_27)
- net PB7: now also J2.28 (Pin_28)
- net PB8: now also J2.29 (Pin_29)
- net PB9: now also J2.30 (Pin_30)
- net PC0: now also J1.10 (Pin_10)
- net PC1: now also J1.9 (Pin_9)
- net PC10: now also J2.13 (Pin_13)
- net PC11: now also J2.14 (Pin_14)
- net PC12: now also J2.15 (Pin_15)
- net PC13: now also J1.12 (Pin_12)
- net PC2: now also J1.8 (Pin_8)
- net PC3: now also J1.7 (Pin_7)
- net PC4: now also J3.27 (Pin_27)
- net PC5: now also J3.26 (Pin_26)
- net PC6: now also J2.1 (Pin_1)
- net PC7: now also J2.2 (Pin_2)
- net PC8: now also J2.3 (Pin_3)
- net PC9: now also J2.4 (Pin_4)
- net PD0: now also J2.16 (Pin_16)
- net PD1: now also J2.17 (Pin_17)
- net PD10: now also J3.6 (Pin_6)
- net PD11: now also J3.5 (Pin_5)
- net PD12: now also J3.4 (Pin_4)
- net PD13: now also J3.3 (Pin_3)
- net PD14: now also J3.2 (Pin_2)
- net PD15: now also J3.1 (Pin_1)
- net PD2: now also J2.18 (Pin_18)
- net PD3: now also J2.19 (Pin_19)
- net PD4: now also J2.20 (Pin_20)
- net PD5: now also J2.21 (Pin_21)
- net PD6: now also J2.22 (Pin_22)
- net PD7: now also J2.23 (Pin_23)
- net PD8: now also J3.8 (Pin_8)
- net PD9: now also J3.7 (Pin_7)
- net PE0: now also J2.31 (Pin_31)
- net PE1: now also J2.32 (Pin_32)
- net PE10: now also J3.19 (Pin_19)
- net PE11: now also J3.18 (Pin_18)
- net PE12: now also J3.17 (Pin_17)
- net PE13: now also J3.16 (Pin_16)
- net PE14: now also J3.15 (Pin_15)
- net PE15: now also J3.14 (Pin_14)
- net PE2: now also J1.18 (Pin_18)
- net PE3: now also J1.17 (Pin_17)
- net PE4: now also J1.16 (Pin_16)
- net PE5: now also J1.15 (Pin_15)
- net PE6: now also J1.14 (Pin_14)
- net PE7: now also J3.22 (Pin_22)
- net PE8: now also J3.21 (Pin_21)
- net PE9: now also J3.20 (Pin_20)
- net PH2: now also J1.13 (Pin_13)
- net VCC_3.3V: now also C23.2, C24.2, J2.33 (Pin_33), J8.1 (Pin_1), J8.2 (Pin_2), J8.3 (Pin_3), J8.4 (Pin_4)
- net VCC_5V: now also J5.1 (Pin_1), J5.2 (Pin_2), J5.3 (Pin_3), J5.4 (Pin_4), J5.5 (Pin_5), J5.6 (Pin_6), J5.7 (Pin_7), J5.8 (Pin_8)
- net VREFH: now also J1.5 (Pin_5)
- net at Y2.1: no longer U2.13 (PH1/XTAL_OUT)
- net at Y2.3: no longer U2.12 (PH0/XTAL_IN)
Other:
- note added: "3.3V & 5V 输出接口"
- note removed: "5V 输出接口"
- moved on the sheet: C1, C10, C11, C12, C13, C14, C17, C18, C2, C20, C21, C22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

Commit message: update
Parts:
- removed J10: Conn_01x25_Pin, symbol Connector:Conn_01x25_Pin
- removed J5, J6: Conn_01x08_Pin, symbol Connector:Conn_01x08_Pin
- removed J7: Conn_01x04_Pin, Connector_PinHeader_2.54mm:PinHeader_1x04_P2.54mm_Vertical, symbol Connector:Conn_01x04_Pin
- removed J8: Conn_01x04_Pin, Connector:FanPinHeader_1x03_P2.54mm_Vertical, symbol Connector:Conn_01x04_Pin
- removed J9: Conn_01x04_Pin, symbol Connector:Conn_01x04_Pin
- added J5, J6: Conn_01x06_Pin, Connector_PinHeader_2.54mm:PinHeader_1x06_P2.54mm_Vertical, symbol Connector:Conn_01x06_Pin
- added J7, J8, J9: Conn_01x05_Pin, Connector_PinHeader_2.54mm:PinHeader_1x05_P2.54mm_Vertical, symbol Connector:Conn_01x05_Pin
- J1: footprint (none) -> Connector_PinHeader_2.54mm:PinHeader_1x18_P2.54mm_Vertical
- J2, J3: footprint (none) -> Connector_PinHeader_2.54mm:PinHeader_1x34_P2.54mm_Vertical
Connections:
- net GND: now also J6.1 (Pin_1), J6.2 (Pin_2), J6.3 (Pin_3), J6.4 (Pin_4), J6.5 (Pin_5), J6.6 (Pin_6), J7.1 (Pin_1), J9.1 (Pin_1), J9.2 (Pin_2), J9.3 (Pin_3), J9.4 (Pin_4), J9.5 (Pin_5)
- net NRST: now also J7.4 (Pin_4)
- net PA13/JTMS_SWDIO: now also J7.3 (Pin_3)
- net PA14/JTCK_SWCLK: now also J7.2 (Pin_2)
- net VCC_3.3V: now also J7.5 (Pin_5), J8.1 (Pin_1), J8.2 (Pin_2), J8.3 (Pin_3), J8.4 (Pin_4), J8.5 (Pin_5)
- net VCC_5V: now also J5.1 (Pin_1), J5.2 (Pin_2), J5.3 (Pin_3), J5.4 (Pin_4), J5.5 (Pin_5), J5.6 (Pin_6)
- net at Y2.1: now also U2.13 (PH1/XTAL_OUT)
- net at Y2.3: now also U2.12 (PH0/XTAL_IN)
Other:
- moved on the sheet: C14, C18, R6, R7, Y2

Commit message: update
Parts:
- removed J5, J6: Conn_01x06_Pin, Connector_PinHeader_2.54mm:PinHeader_1x06_P2.54mm_Vertical, symbol Connector:Conn_01x06_Pin
- removed J8, J9: Conn_01x05_Pin, Connector_PinHeader_2.54mm:PinHeader_1x05_P2.54mm_Vertical, symbol Connector:Conn_01x05_Pin
- added J5, J6, J8, J9: Conn_01x04_Pin, Connector_PinHeader_2.54mm:PinHeader_1x04_P2.54mm_Vertical, symbol Connector:Conn_01x04_Pin
Connections:
- net GND: now also J6.1 (Pin_1), J6.2 (Pin_2), J6.3 (Pin_3), J6.4 (Pin_4), J9.1 (Pin_1), J9.2 (Pin_2), J9.3 (Pin_3), J9.4 (Pin_4)
- net VCC_3.3V: now also J8.1 (Pin_1), J8.2 (Pin_2), J8.3 (Pin_3), J8.4 (Pin_4)
- net VCC_5V: now also J5.1 (Pin_1), J5.2 (Pin_2), J5.3 (Pin_3), J5.4 (Pin_4)

Commit message: update
Connections:
- net NRST: now also J7.2 (Pin_2); no longer J7.4 (Pin_4)
- net PA13/JTMS_SWDIO: now also J7.4 (Pin_4); no longer J7.3 (Pin_3)
- net PA14/JTCK_SWCLK: now also J7.3 (Pin_3); no longer J7.2 (Pin_2)
Other:
- moved on the sheet: R6, R7
Changed lines of the file:
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@@
 	)
 	(junction
-		(at 313.69 203.2)
+		(at 313.69 205.74)
 		(diameter 0)
 		(color 0 0 0 0)
@@
 	)
 	(junction
-		(at 313.69 205.74)
+		(at 313.69 208.28)
 		(diameter 0)
 		(color 0 0 0 0)
@@
 	(wire
 		(pts
-			(xy 288.29 203.2) (xy 313.69 203.2)
+			(xy 288.29 205.74) (xy 313.69 205.74)
 		)
 		(stroke
@@
 	(wire
 		(pts
+			(xy 288.29 203.2) (xy 300.99 203.2)
+		)
+		(stroke
+			(width 0)
+			(type default)
+		)
+	)
+	(wire
+		(pts
 			(xy 330.2 114.3) (xy 327.66 114.3)
 		)
@@
 	(wire
 		(pts
-			(xy 313.69 203.2) (xy 322.58 203.2)
+			(xy 313.69 205.74) (xy 322.58 205.74)
 		)
 		(stroke
@@
 	(wire
 		(pts
-			(xy 313.69 213.36) (xy 321.31 213.36)
+			(xy 313.69 215.9) (xy 321.31 215.9)
 		)
 		(stroke
@@
 	(wire
 		(pts
-			(xy 288.29 208.28) (xy 292.1 208.28)
+			(xy 288.29 208.28) (xy 313.69 208.28)
 		)
 		(stroke
@@
 	(wire
 		(pts
-			(xy 288.29 205.74) (xy 313.69 205.74)
-		)
-		(stroke
-			(width 0)
-			(type default)
-		)
-	)
-	(wire
-		(pts
 			(xy 203.2 60.96) (xy 213.36 60.96)
 		)
@@
 	(wire
 		(pts
-			(xy 313.69 195.58) (xy 323.85 195.58)
+			(xy 313.69 198.12) (xy 323.85 198.12)
 		)
 		(stroke
@@
 	(wire
 		(pts
-			(xy 313.69 205.74) (xy 322.58 205.74)
+			(xy 313.69 208.28) (xy 322.58 208.28)
 		)
 		(stroke
@@
 	)
 	(label "NRST"
-		(at 292.1 208.28 0)
+		(at 300.99 203.2 0)
 		(fields_autoplaced yes)
 		(effects
@@
 	)
 	(label "PA13{slash}JTMS_SWDIO"
-		(at 322.58 205.74 0)
+		(at 322.58 208.28 0)
 		(fields_autoplaced yes)
 		(effects
@@
 	)
 	(label "PA14{slash}JTCK_SWCLK"
-		(at 322.58 203.2 0)
+		(at 322.58 205.74 0)
 		(fields_autoplaced yes)
 		(effects
@@
 	(symbol
 		(lib_id "Device:R")
-		(at 313.69 209.55 0)
+		(at 313.69 212.09 0)
 		(unit 1)
 		(exclude_from_sim no)
@@
 		(dnp no)
 		(property "Reference" "R7"
-			(at 316.23 208.2799 0)
+			(at 316.23 210.8199 0)
 			(effects
 				(font
@@
 		)
 		(property "Value" "10K"
-			(at 313.944 211.074 90)
+			(at 313.944 213.614 90)
 			(effects
 				(font
@@
 		)
 		(property "Footprint" "Resistor_SMD:R_0603_1608Metric"
-			(at 311.912 209.55 90)
+			(at 311.912 212.09 90)
 			(effects
 				(font
@@
 		)
 		(property "Datasheet" "~"
-			(at 313.69 209.55 0)
+			(at 313.69 212.09 0)
 			(effects
 				(font
@@
 		)
 		(property "Description" "Resistor"
-			(at 313.69 209.55 0)
+			(at 313.69 212.09 0)
 			(effects
 				(font
@@
 	(symbol
 		(lib_id "Device:R")
-		(at 313.69 199.39 0)
+		(at 313.69 201.93 0)
 		(unit 1)
 		(exclude_from_sim no)
@@
 		(dnp no)
 		(property "Reference" "R6"
-			(at 316.23 198.1199 0)
+			(at 316.23 200.6599 0)
 			(effects
 				(font
@@
 		)
 		(property "Value" "10K"
-			(at 313.944 200.914 90)
+			(at 313.944 203.454 90)
 			(effects
 				(font
@@
 		)
 		(property "Footprint" "Resistor_SMD:R_0603_1608Metric"
-			(at 311.912 199.39 90)
+			(at 311.912 201.93 90)
 			(effects
 				(font
@@
 		)
 		(property "Datasheet" "~"
-			(at 313.69 199.39 0)
+			(at 313.69 201.93 0)
 			(effects
 				(font
@@
 		)
 		(property "Description" "Resistor"
-			(at 313.69 199.39 0)
+			(at 313.69 201.93 0)
 			(effects
 				(font
@@
 	(symbol
 		(lib_id "power:VCC")
-		(at 321.31 213.36 270)
+		(at 321.31 215.9 270)
 		(unit 1)
 		(exclude_from_sim no)
@@
 		(dnp no)
 		(property "Reference" "#PWR051"
-			(at 317.5 213.36 0)
+			(at 317.5 215.9 0)
 			(effects
 				(font
@@
 		)
 		(property "Value" "VCC_3.3V"
-			(at 324.612 213.36 90)
+			(at 324.612 215.9 90)
 			(effects
 				(font
@@
 		)
 		(property "Footprint" ""
-			(at 321.31 213.36 0)
+			(at 321.31 215.9 0)
 			(effects
 				(font
@@
 		)
 		(property "Datasheet" ""
-			(at 321.31 213.36 0)
+			(at 321.31 215.9 0)
 			(effects
 				(font
@@
 		)
 		(property "Description" "Power symbol creates a global label with name \"VCC\""
-			(at 321.31 213.36 0)
+			(at 321.31 215.9 0)
 			(effects
 				(font
@@
 	(symbol
 		(lib_id "power:VCC")
-		(at 323.85 195.58 270)
+		(at 323.85 198.12 270)
 		(unit 1)
 		(exclude_from_sim no)
@@
 		(dnp no)
 		(property "Reference" "#PWR052"
-			(at 320.04 195.58 0)
+			(at 320.04 198.12 0)
 			(effects
 				(font
@@
 		)
 		(property "Value" "VCC_3.3V"
-			(at 327.152 195.58 90)
+			(at 327.152 198.12 90)
 			(effects
 				(font
@@
 		)
 		(property "Footprint" ""
-			(at 323.85 195.58 0)
+			(at 323.85 198.12 0)
 			(effects
 				(font
@@
 		)
 		(property "Datasheet" ""
-			(at 323.85 195.58 0)
+			(at 323.85 198.12 0)
 			(effects
 				(font
@@
 		)
 		(property "Description" "Power symbol creates a global label with name \"VCC\""
-			(at 323.85 195.58 0)
+			(at 323.85 198.12 0)
 			(effects
 				(font

Commit message: update
Parts:
- removed J7: Conn_01x05_Pin, Connector_PinHeader_2.54mm:PinHeader_1x05_P2.54mm_Vertical, symbol Connector:Conn_01x05_Pin
- added J7: Conn_01x04_Pin, Connector_PinHeader_2.54mm:PinHeader_1x04_P2.54mm_Vertical, symbol Connector:Conn_01x04_Pin
Connections:
- net GND: now also J7.1 (Pin_1)
- net NRST: now also SW1.1, SW1.2
- net PA13/JTMS_SWDIO: now also J7.3 (Pin_3)
- net PA14/JTCK_SWCLK: now also J7.2 (Pin_2)
- net VCC_3.3V: now also J7.4 (Pin_4); no longer SW1.1, SW1.2
Other:
- moved on the sheet: C13, R5, SW1

Commit message: update
Parts:
- removed J4: MD, Connector_PinHeader_2.54mm:PinHeader_1x02_P2.54mm_Vertical, symbol Connector:Conn_01x02_Pin
- added J10: Conn_01x03_Pin, Connector_PinHeader_2.54mm:PinHeader_1x03_P2.54mm_Vertical, symbol Connector:Conn_01x03_Pin
Connections:
- net GND: now also J10.2 (Pin_2), J10.3 (Pin_3)
- net PB11/MD: now also J10.1 (Pin_1)
Changed lines of the file:
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@@
 	(title_block
 		(title "UINIO-MCU-HC32F460PETB")
-		(date "2024-08-12")
+		(date "2024-08-20")
 		(rev "Version 1.0.0")
 		(company "UinIO.com 电子技术实验室")
@@
 	)
 	(junction
+		(at 199.39 55.88)
+		(diameter 0)
+		(color 0 0 0 0)
+	)
+	(junction
 		(at 233.68 228.6)
 		(diameter 0)
@@
 	(wire
 		(pts
+			(xy 199.39 53.34) (xy 199.39 55.88)
+		)
+		(stroke
+			(width 0)
+			(type default)
+		)
+	)
+	(wire
+		(pts
 			(xy 330.2 152.4) (xy 330.2 149.86)
 		)
@@
 	(wire
 		(pts
+			(xy 199.39 55.88) (xy 198.12 55.88)
+		)
+		(stroke
+			(width 0)
+			(type default)
+		)
+	)
+	(wire
+		(pts
 			(xy 340.36 60.96) (xy 330.2 60.96)
 		)
@@
 	(wire
 		(pts
+			(xy 200.66 55.88) (xy 199.39 55.88)
+		)
+		(stroke
+			(width 0)
+			(type default)
+		)
+	)
+	(wire
+		(pts
 			(xy 66.04 210.82) (xy 68.58 210.82)
 		)
@@
 	(wire
 		(pts
-			(xy 200.66 53.34) (xy 198.12 53.34)
+			(xy 199.39 53.34) (xy 198.12 53.34)
 		)
 		(stroke
@@
 	(symbol
 		(lib_id "power:GND")
-		(at 200.66 53.34 90)
+		(at 200.66 55.88 90)
 		(unit 1)
 		(exclude_from_sim no)
@@
 		(dnp no)
 		(property "Reference" "#PWR030"
-			(at 207.01 53.34 0)
+			(at 207.01 55.88 0)
 			(effects
 				(font
@@
 		)
 		(property "Value" "GND"
-			(at 203.454 53.594 90)
+			(at 203.454 56.134 90)
 			(effects
 				(font
@@
 		)
 		(property "Footprint" ""
-			(at 200.66 53.34 0)
+			(at 200.66 55.88 0)
 			(effects
 				(font
@@
 		)
 		(property "Datasheet" ""
-			(at 200.66 53.34 0)
+			(at 200.66 55.88 0)
 			(effects
 				(font
@@
 		)
 		(property "Description" "Power symbol creates a global label with name \"GND\" , ground"
-			(at 200.66 53.34 0)
+			(at 200.66 55.88 0)
 			(effects
 				(font
@@
 	)
 	(symbol
+		(lib_id "Connector:Conn_01x03_Pin")
+		(at 193.04 53.34 0)
+		(unit 1)
+		(exclude_from_sim no)
+		(in_bom yes)
+		(on_board yes)
+		(dnp no)
+		(property "Reference" "J10"
+			(at 196.088 46.99 0)
+			(effects
+				(font
+					(size 1.27 1.27)
+				)
+			)
+		)
+		(property "Value" "Conn_01x03_Pin"
+			(at 185.42 53.34 0)
+			(effects
+				(font
+					(size 1.27 1.27)
+				)
+			)
+		)
+		(property "Footprint" "Connector_PinHeader_2.54mm:PinHeader_1x03_P2.54mm_Vertical"
+			(at 193.04 53.34 0)
+			(effects
+				(font
+					(size 1.27 1.27)
+				)
+				(hide yes)
+			)
+		)
+		(property "Datasheet" "~"
+			(at 193.04 53.34 0)
+			(effects
+				(font
+					(size 1.27 1.27)
+				)
+				(hide yes)
+			)
+		)
+		(property "Description" "Generic connector, single row, 01x03, script generated"
+			(at 193.04 53.34 0)
+			(effects
+				(font
+					(size 1.27 1.27)
+				)
+				(hide yes)
+			)
+		)
+		(pin "3"
+		)
+		(pin "2"
+		)
+		(pin "1"
+		)
+		(instances
+			(project ""
+				(path "/6fcf9576-1508-4150-862c-de9a7b38786e"
+					(reference "J10")
+					(unit 1)
+				)
+			)
+		)
+	)
+	(symbol
 		(lib_id "power:VCC")
 		(at 139.7 137.16 90)
@@
 					(unit 1)
 				)
-			)
-		)
-	)
-	(symbol
-		(lib_id "Connector:Conn_01x02_Pin")
-		(at 193.04 50.8 0)
-		(unit 1)
-		(exclude_from_sim no)
-		(in_bom yes)
-		(on_board yes)
-		(dnp no)
-		(property "Reference" "J4"
-			(at 195.834 46.99 0)
-			(effects
-				(font
-					(size 1.27 1.27)
-				)
-			)
-		)
-		(property "Value" "MD"
-			(at 196.088 55.626 0)
-			(effects
-				(font
-					(size 1.27 1.27)
-				)
-			)
-		)
-		(property "Footprint" "Connector_PinHeader_2.54mm:PinHeader_1x02_P2.54mm_Vertical"
-			(at 193.04 50.8 0)
-			(effects
-				(font
-					(size 1.27 1.27)
-				)
-				(hide yes)
-			)
-		)
-		(property "Datasheet" "~"
-			(at 193.04 50.8 0)
-			(effects
-				(font
-					(size 1.27 1.27)
-				)
-				(hide yes)
-			)
-		)
-		(property "Description" "Generic connector, single row, 01x02, script generated"
-			(at 193.04 50.8 0)
-			(effects
-				(font
-					(size 1.27 1.27)
-				)
-				(hide yes)
-			)
-		)
-		(pin "1"
-		)
-		(pin "2"
-		)
-		(instances
-			(project ""
-				(path "/6fcf9576-1508-4150-862c-de9a7b38786e"
-					(reference "J4")
-					(unit 1)
-				)

Commit message: update
Parts:
- renumbered J10 to J4
Changed lines of the file:
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@@
 		(on_board yes)
 		(dnp no)
-		(property "Reference" "J10"
+		(property "Reference" "J4"
 			(at 196.088 46.99 0)
 			(effects
@@
 			(project ""
 				(path "/6fcf9576-1508-4150-862c-de9a7b38786e"
-					(reference "J10")
+					(reference "J4")
 					(unit 1)
 				)
