File: UINIO-MCU-HC32F460PETB.kicad_sch (KiCad schematic)
At the start: 51 parts, among them J1 Conn_01x18_Pin, J2 Conn_01x34_Pin, J3 Conn_01x34_Pin, J4 Conn_01x03_Pin, J5 Conn_01x04_Pin, J6 Conn_01x04_Pin, J7 Conn_01x04_Pin, J8 Conn_01x04_Pin, J9 Conn_01x04_Pin, SW1 NRST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

Commit message: update
Parts:
- added F1: Fuse, Fuse:Fuse_1206_3216Metric, symbol Device:Fuse
Connections:
- net VCC_5V: now also F1.2; no longer J5.1 (Pin_1), J5.2 (Pin_2), J5.3 (Pin_3), J5.4 (Pin_4)
- new net: F1.1, J5.1 (Pin_1), J5.2 (Pin_2), J5.3 (Pin_3), J5.4 (Pin_4)
Changed lines of the file:
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@@
 	(wire
 		(pts
+			(xy 229.87 199.39) (xy 234.95 199.39)
+		)
+		(stroke
+			(width 0)
+			(type default)
+		)
+	)
+	(wire
+		(pts
 			(xy 152.4 78.74) (xy 152.4 83.82)
 		)
@@
 	(wire
 		(pts
-			(xy 217.17 199.39) (xy 234.95 199.39)
+			(xy 217.17 199.39) (xy 222.25 199.39)
 		)
 		(stroke
@@
 					(unit 1)
 				)
+			)
+		)
+	)
+	(symbol
+		(lib_id "Device:Fuse")
+		(at 226.06 199.39 90)
+		(unit 1)
+		(exclude_from_sim no)
+		(in_bom yes)
+		(on_board yes)
+		(dnp no)
+		(property "Reference" "F1"
+			(at 226.06 195.072 90)
+			(effects
+				(font
+					(size 1.27 1.27)
+				)
+			)
+		)
+		(property "Value" "Fuse"
+			(at 226.06 197.104 90)
+			(effects
+				(font
+					(size 1.27 1.27)
+				)
+			)
+		)
+		(property "Footprint" "Fuse:Fuse_1206_3216Metric"
+			(at 226.06 201.168 90)
+			(effects
+				(font
+					(size 1.27 1.27)
+				)
+				(hide yes)
+			)
+		)
+		(property "Datasheet" "~"
+			(at 226.06 199.39 0)
+			(effects
+				(font
+					(size 1.27 1.27)
+				)
+				(hide yes)
+			)
+		)
+		(property "Description" "Fuse"
+			(at 226.06 199.39 0)
+			(effects
+				(font
+					(size 1.27 1.27)
+				)
+				(hide yes)
+			)
+		)
+		(pin "1"
+		)
+		(pin "2"
+		)
+		(instances
+			(project ""
+				(path "/6fcf9576-1508-4150-862c-de9a7b38786e"
+					(reference "F1")
+					(unit 1)
+				)

Commit message: update
Connections:
- net GND: now also J7.2 (Pin_2); no longer J7.1 (Pin_1)
- net PA13/JTMS_SWDIO: now also J7.4 (Pin_4); no longer J7.3 (Pin_3)
- net PA14/JTCK_SWCLK: now also J7.3 (Pin_3); no longer J7.2 (Pin_2)
- net VCC_3.3V: now also J7.1 (Pin_1); no longer J7.4 (Pin_4)
Other:
- moved on the sheet: R6, R7
Changed lines of the file:
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@@
 	)
 	(junction
-		(at 313.69 205.74)
+		(at 313.69 208.28)
 		(diameter 0)
 		(color 0 0 0 0)
@@
 	)
 	(junction
-		(at 313.69 208.28)
+		(at 313.69 210.82)
 		(diameter 0)
 		(color 0 0 0 0)
@@
 	(wire
 		(pts
-			(xy 288.29 205.74) (xy 313.69 205.74)
+			(xy 288.29 208.28) (xy 313.69 208.28)
 		)
 		(stroke
@@
 	(wire
 		(pts
-			(xy 313.69 205.74) (xy 322.58 205.74)
+			(xy 313.69 208.28) (xy 322.58 208.28)
 		)
 		(stroke
@@
 	(wire
 		(pts
-			(xy 289.56 210.82) (xy 288.29 210.82)
-		)
-		(stroke
-			(width 0)
-			(type default)
-		)
-	)
-	(wire
-		(pts
 			(xy 218.44 228.6) (xy 220.98 228.6)
 		)
@@
 	(wire
 		(pts
-			(xy 289.56 203.2) (xy 288.29 203.2)
+			(xy 290.83 205.74) (xy 288.29 205.74)
 		)
 		(stroke
@@
 	(wire
 		(pts
-			(xy 313.69 215.9) (xy 321.31 215.9)
+			(xy 313.69 218.44) (xy 321.31 218.44)
 		)
 		(stroke
@@
 	(wire
 		(pts
-			(xy 288.29 208.28) (xy 313.69 208.28)
+			(xy 288.29 210.82) (xy 313.69 210.82)
 		)
 		(stroke
@@
 	(wire
 		(pts
+			(xy 288.29 203.2) (xy 290.83 203.2)
+		)
+		(stroke
+			(width 0)
+			(type default)
+		)
+	)
+	(wire
+		(pts
 			(xy 316.23 101.6) (xy 321.31 101.6)
 		)
@@
 	(wire
 		(pts
-			(xy 313.69 198.12) (xy 323.85 198.12)
+			(xy 313.69 200.66) (xy 323.85 200.66)
 		)
 		(stroke
@@
 	(wire
 		(pts
-			(xy 313.69 208.28) (xy 322.58 208.28)
+			(xy 313.69 210.82) (xy 322.58 210.82)
 		)
 		(stroke
@@
 	)
 	(label "PA13{slash}JTMS_SWDIO"
-		(at 322.58 208.28 0)
+		(at 322.58 210.82 0)
 		(fields_autoplaced yes)
 		(effects
@@
 	)
 	(label "PA14{slash}JTCK_SWCLK"
-		(at 322.58 205.74 0)
+		(at 322.58 208.28 0)
 		(fields_autoplaced yes)
 		(effects
@@
 	(symbol
 		(lib_id "Device:R")
-		(at 313.69 212.09 0)
+		(at 313.69 214.63 0)
 		(unit 1)
 		(exclude_from_sim no)
@@
 		(dnp no)
 		(property "Reference" "R7"
-			(at 316.23 210.8199 0)
+			(at 316.23 213.3599 0)
 			(effects
 				(font
@@
 		)
 		(property "Value" "10K"
-			(at 313.944 213.614 90)
+			(at 313.944 216.154 90)
 			(effects
 				(font
@@
 		)
 		(property "Footprint" "Resistor_SMD:R_0603_1608Metric"
-			(at 311.912 212.09 90)
+			(at 311.912 214.63 90)
 			(effects
 				(font
@@
 		)
 		(property "Datasheet" "~"
-			(at 313.69 212.09 0)
+			(at 313.69 214.63 0)
 			(effects
 				(font
@@
 		)
 		(property "Description" "Resistor"
-			(at 313.69 212.09 0)
+			(at 313.69 214.63 0)
 			(effects
 				(font
@@
 	(symbol
 		(lib_id "Device:R")
-		(at 313.69 201.93 0)
+		(at 313.69 204.47 0)
 		(unit 1)
 		(exclude_from_sim no)
@@
 		(dnp no)
 		(property "Reference" "R6"
-			(at 316.23 200.6599 0)
+			(at 316.23 203.1999 0)
 			(effects
 				(font
@@
 		)
 		(property "Value" "10K"
-			(at 313.944 203.454 90)
+			(at 313.944 205.994 90)
 			(effects
 				(font
@@
 		)
 		(property "Footprint" "Resistor_SMD:R_0603_1608Metric"
-			(at 311.912 201.93 90)
+			(at 311.912 204.47 90)
 			(effects
 				(font
@@
 		)
 		(property "Datasheet" "~"
-			(at 313.69 201.93 0)
+			(at 313.69 204.47 0)
 			(effects
 				(font
@@
 		)
 		(property "Description" "Resistor"
-			(at 313.69 201.93 0)
+			(at 313.69 204.47 0)
 			(effects
 				(font
@@
 	(symbol
 		(lib_id "power:GND")
-		(at 289.56 203.2 90)
+		(at 290.83 205.74 90)
 		(unit 1)
 		(exclude_from_sim no)
@@
 		(dnp no)
 		(property "Reference" "#PWR06"
-			(at 295.91 203.2 0)
+			(at 297.18 205.74 0)
 			(effects
 				(font
@@
 		)
 		(property "Value" "GND"
-			(at 294.64 203.2 90)
+			(at 295.91 205.74 90)
 			(effects
 				(font
@@
 		)
 		(property "Footprint" ""
-			(at 289.56 203.2 0)
+			(at 290.83 205.74 0)
 			(effects
 				(font
@@
 		)
 		(property "Datasheet" ""
-			(at 289.56 203.2 0)
+			(at 290.83 205.74 0)
 			(effects
 				(font
@@
 		)
 		(property "Description" "Power symbol creates a global label with name \"GND\" , ground"
-			(at 289.56 203.2 0)
+			(at 290.83 205.74 0)
 			(effects
 				(font
@@
 	(symbol
 		(lib_id "power:VCC")
-		(at 289.56 210.82 270)
+		(at 290.83 203.2 270)
 		(unit 1)
 		(exclude_from_sim no)
@@
 		(dnp no)
 		(property "Reference" "#PWR047"
-			(at 285.75 210.82 0)
+			(at 287.02 203.2 0)
 			(effects
 				(font
@@
 		)
 		(property "Value" "VCC_3.3V"
-			(at 292.862 210.82 90)
+			(at 294.132 203.2 90)
 			(effects
 				(font
@@
 		)
 		(property "Footprint" ""
-			(at 289.56 210.82 0)
+			(at 290.83 203.2 0)
 			(effects
 				(font
@@
 		)
 		(property "Datasheet" ""
-			(at 289.56 210.82 0)
+			(at 290.83 203.2 0)
 			(effects
 				(font
@@
 		)
 		(property "Description" "Power symbol creates a global label with name \"VCC\""
-			(at 289.56 210.82 0)
+			(at 290.83 203.2 0)
 			(effects
 				(font
@@
 	(symbol
 		(lib_id "power:VCC")
-		(at 321.31 215.9 270)
+		(at 321.31 218.44 270)
 		(unit 1)
 		(exclude_from_sim no)
@@
 		(dnp no)
 		(property "Reference" "#PWR051"
-			(at 317.5 215.9 0)
+			(at 317.5 218.44 0)
 			(effects
 				(font
@@
 		)
 		(property "Value" "VCC_3.3V"
-			(at 324.612 215.9 90)
+			(at 324.612 218.44 90)
 			(effects
 				(font
@@
 		)
 		(property "Footprint" ""
-			(at 321.31 215.9 0)
+			(at 321.31 218.44 0)
 			(effects
 				(font
@@
 		)
 		(property "Datasheet" ""
-			(at 321.31 215.9 0)
+			(at 321.31 218.44 0)
 			(effects
 				(font
@@
 		)
 		(property "Description" "Power symbol creates a global label with name \"VCC\""
-			(at 321.31 215.9 0)
+			(at 321.31 218.44 0)
 			(effects
 				(font
@@
 	(symbol
 		(lib_id "power:VCC")
-		(at 323.85 198.12 270)
+		(at 323.85 200.66 270)
 		(unit 1)
 		(exclude_from_sim no)
@@
 		(dnp no)
 		(property "Reference" "#PWR052"
-			(at 320.04 198.12 0)
+			(at 320.04 200.66 0)
 			(effects
 				(font
@@
 		)
 		(property "Value" "VCC_3.3V"
-			(at 327.152 198.12 90)
+			(at 327.152 200.66 90)
 			(effects
 				(font
@@
 		)
 		(property "Footprint" ""
-			(at 323.85 198.12 0)
+			(at 323.85 200.66 0)
 			(effects
 				(font
@@
 		)
 		(property "Datasheet" ""
-			(at 323.85 198.12 0)
+			(at 323.85 200.66 0)
 			(effects
 				(font
@@
 		)
 		(property "Description" "Power symbol creates a global label with name \"VCC\""
-			(at 323.85 198.12 0)
+			(at 323.85 200.66 0)
 			(effects
 				(font
